File: kicad-project/eth01-24v/eth01-24v.kicad_sch (KiCad schematic)
At the start: 4 parts, among them U1 WT32-ETH01, U2 XL-6009-ADJ

Commit message: ajout photos et première version pcb
Parts:
- removed U2: XL-6009-ADJ, esp32-24v-io:XL6009_module_SMT, symbol Regulator_Switching:XL1509-ADJ
- removed U3: ~, WT32-ETH01:OP71A04, symbol WT32-ETH01:OP71A04-3.3V-24v
- added BSS1: ~, WT32-ETH01:BSS138, symbol WT32-ETH01:BSS138-LevelShifterBoard
- added J1, J10, J11, J12, J9: KF301-2P, WT32-ETH01:KF3012P, symbol WT32-ETH01:KF301-2P
- added J13, J2, J3, J4, J5, J6, J7, J8: KF301-3P, KF3013P, symbol WT32-ETH01:KF301-3P
- added U2: ~, WT32-ETH01:MCP23017, symbol WT32-ETH01:MCP23017-CJMCU2317
- added U3: ~, WT32-ETH01:OP71A04, symbol WT32-ETH01:OP71A04-24v-3.3v
- added U5, U7: ~, WT32-ETH01:OP71A04, symbol Boards:OP71A04-3.3V-24v
- added U8: ~, WT32-ETH01:MP1584_AIO, symbol WT32-ETH01:MP1584
- U1: github (none) -> https://github.com/egnor/wt32-eth01
Connections:
- net +24V: now also J1.1, J1.2, J12.2, J9.1, U5.9 (Vcc), U7.9 (Vcc), U8.1 (IN-), U8.2 (IN-)
- net GND: now also U1.23 (GND), BSS1.10 (GND), BSS1.4 (GND), J10.1, J12.1, J13.2, J4.3, J7.1, J8.1, J8.3, U2.21 (GND), U2.9 (GND), U3.10 (Ground), U3.2 (1-), U3.4 (2-), U3.6 (3-), U3.8 (4-), U5.10 (Ground), U5.2 (1-), U5.4 (2-), U5.6 (3-), U5.8 (4-), U7.10 (Ground), U7.2 (1-), U7.4 (2-), U7.6 (3-), U7.8 (4-), U8.5 (OUT-), U8.6 (OUT-)
- net at U4.11 (O1): now also U2.20 (B7); no longer U1.22 (IO39/ADC1_CH3/INPUT_ONLY)
- net at U4.12 (O2): now also U2.19 (B6); no longer U1.21 (IO36/ADC1_CH0/INPUT_ONLY)
- net at U4.13 (O3): now also U2.18 (B5); no longer U1.20 (IO15/ADC2_CH3/TCH3)
- net at U4.14 (O4): now also U2.17 (B4); no longer U1.19 (IO14/ADC2_CH6/TCH6)
- net 3.3V: now reaches U1.10 (3.3V), U1.3 (3.3V), U4.9 (Vcc)
- net 3.3V: now also BSS1.3 (LV), U2.10 (VCC), U2.11 (VCC), U3.9 (Vcc)
- net SCL: now reaches U1.5 (IO32/ADC1_CH4/TCH9)
- net SCL: now also U2.8 (SCL/SCK)
- net SDA: now reaches U1.6 (IO33/ADC1_CH5/TCH8)
- net SDA: now also U2.7 (SDA/SI)
- net 5V: now reaches U1.12 (5V)
- net 5V: now also U8.7 (OUT+), U8.8 (OUT+)
- net at U1.16 (IO4/ADC2_CH0/TCH0): now also BSS1.5 (LV3)
- net IN1-24V renamed E-STOP
- net E-STOP: now also J10.2, J2.3
- net IN2-24V renamed SIGNAL
- net SIGNAL: now also J2.2, J9.2
- net IN3-24V: no longer names the net of U4.5 (3+)
- net IN3-24V: now also J2.1
- net IN4-24V: no longer names the net of U4.7 (4+)
- net IN4-24V: now also J3.3
- new net: J11.1, J11.2, U8.3 (IN+), U8.4 (IN+)
- new net: J3.2, U3.1 (1+)
- new net: U2.16 (B3), U3.11 (O1)
- new net: U2.15 (B2), U3.12 (O2)
- new net: U2.14 (B1), U3.13 (O3)
- new net: U2.13 (B0), U3.14 (O4)
- new net: J3.1, U3.3 (2+)
- new net: J7.3, U3.5 (3+)
- new net: J7.2, U3.7 (4+)
- new net: U2.23 (A0), U5.1 (1+)
- new net: U2.24 (A1), U5.3 (2+)
- new net: U2.25 (A2), U5.5 (3+)
- new net: U2.26 (A3), U5.7 (4+)
- new net: U2.27 (A4), U7.1 (1+)
- new net: U2.28 (A5), U7.3 (2+)
- new net: U2.29 (A6), U7.5 (3+)
- new net: U2.30 (A7), U7.7 (4+)
- new net: J5.2, U7.11 (O1)
- new net: J5.3, U7.12 (O2)
- new net: J4.1, U7.13 (O3)
- new net: J4.2, U7.14 (O4)
- new net: BSS1.2 (LV2), U1.19 (IO14/ADC2_CH6/TCH6)
- new net: BSS1.1 (LV1), U1.20 (IO15/ADC2_CH3/TCH3)
- new net: J5.1, U5.14 (O4)
- new net: J6.1, U5.11 (O1)
- new net: J6.2, U5.12 (O2)
- new net: J6.3, U5.13 (O3)
- new net +5V: BSS1.9 (HV)
- new net DIR+: BSS1.8 (HV2), J13.1
- new net EN+: BSS1.7 (HV1), J8.2
- new net InterruptA: U1.21 (IO36/ADC1_CH0/INPUT_ONLY), U2.22 (ITA)
- new net InteruptB: U1.22 (IO39/ADC1_CH3/INPUT_ONLY), U2.12 (ITB)
- new net PUL+: BSS1.11 (HV3), J13.3
- no-connect marks 11 -> 19
Other:
- note added: "0V?"
- note added: "24V"
- note added: "24V plug motor"
- note added: "8 Inputs 24V / 1 GND"
- note added: "8 Outputs 24V / 1 GND"
- note added: "A Faire - Ajouter sonde CNC Z - en 24V avec bornes alimentation - intégrer pins pour la commande moteur - mettre un bus I/O pour avoir plus d'entrées/sorties que juste les pins libres - prévoir soit I/O en 5V soit 24V, soit 3,3V - ajouter l'alimentation sur la board"
- note added: "Alimentation 24V"
- note added: "E-STOP"
- note added: "Motor drive connection DM556"
- note added: "Signal"
- note added: "Sonde Z Mach3"
- note added: "adress bus"
- moved on the sheet: U1

Commit message: routage ok
Parts:
- removed J2: KF301-3P, KF3013P, symbol WT32-ETH01:KF301-3P
- added DRA1, DRA2: DIN_Rail_Adapter, MountingEquipment:DINRailAdapter_3xM3_PhoenixContact_1201578, symbol Mechanical:DIN_Rail_Adapter
- added J2: KF301-2P, WT32-ETH01:KF3012P, symbol WT32-ETH01:KF301-2P
- U3, U4: footprint WT32-ETH01:OP71A04 -> WT32-ETH01:OP71A04 - 24V3.3V
- U5, U7: footprint WT32-ETH01:OP71A04 -> WT32-ETH01:OP71A04 - 3.3V24V
Connections:
- net +5V is gone; now on net 5V: BSS1.9 (HV)
- net +24V: now also J11.1, U8.3 (IN+), U8.4 (IN+); no longer J1.2, U8.1 (IN-), U8.2 (IN-)
- net GND: now also J1.2, J11.2, U8.1 (IN-), U8.2 (IN-), J2.2
- net at U4.5 (3+): now also J2.1
Other:
- note added: "6 Inputs 24V / 2 GND"
- note removed: "0V?"
- note removed: "24V"
- note removed: "8 Inputs 24V / 1 GND"
- note removed: "E-STOP"
- note removed: "Signal"
- moved on the sheet: J1, J11
