File: kicad-project/eth01-24v/eth01-24v.kicad_sch (KiCad schematic)
At the start: 23 parts, among them J1 KF301-2P, J10 KF301-2P, J11 KF301-2P, J12 KF301-2P, J13 KF301-3P, J2 KF301-2P, J3 KF301-3P, J4 KF301-3P, J5 KF301-3P, J6 KF301-3P, J7 KF301-3P, J8 KF301-3P, J9 KF301-2P, U1 WT32-ETH01

Commit message: moteur DM556 optionnel avec broches configurables + numéros GPIO sur le schéma
- Moteur pas-à-pas activable/désactivable depuis l'onglet Configuration I/O,
  avec tableau des broches PUL+/DIR+/EN+ (grisé si moteur désactivé)
- Moteur désactivé : broches libres pour les I/O, pas d'abonnement MQTT motor/*
- Nouvelle API /api/motor/config (GET/POST) avec contrôle des conflits de broches
- Schéma KiCad : ajout des numéros de GPIO

Co-Authored-By: Claude Opus 5.5 <noreply@anthropic.com>
Parts:
- BSS1, U2, U3, U4, U5, U7, U8: value ~ -> (none)
